Commit message: ajout de interpolation

File: real_robot/robot_models/URDF_description/urdf/lynx_ses900_optimized.urdf (robot description, URDF)
Before this commit: robot lynx_ses900, 8 links, 7 joints
Joints:
- joint joint_1: axis 0 0 1 -> 0 0 -1; limit lower=-2.967 upper=2.967 effort=50 velocity=1.5 -> lower=-3.1416 upper=3.1416 effort=50 velocity=1.5
- joint joint_2: limit lower=-2.0 upper=2.0 effort=50 velocity=1.5 -> lower=-3.1416 upper=3.1416 effort=50 velocity=1.5
- joint joint_3: limit lower=-2.0 upper=2.0 effort=40 velocity=1.5 -> lower=-3.1416 upper=3.1416 effort=40 velocity=1.5
- joint joint_4: axis 0 0 1 -> 0 0 -1; limit lower=-2.0 upper=2.0 effort=30 velocity=1.5 -> lower=-3.1416 upper=3.1416 effort=30 velocity=1.5
- joint joint_5: limit lower=-2.0 upper=2.0 effort=20 velocity=1.5 -> lower=-3.1416 upper=3.1416 effort=20 velocity=1.5
